File: SCClimate/SCClimate.sch (KiCad schematic (older format))
At the start: 77 parts, among them J11 HVAC, J3 DISP_SERIAL, J4 SERIAL, J7 PIR, Q1 TEPT5700, Q6 2N6073B, Q7 2N6073B, Q8 2N6073B, SW1 RESET, SW2 MODE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

Commit message: updates
Parts:
- added R? (x2): 180, Resistor_SMD:R_0805_2012Metric_Pad1.20x1.40mm_HandSolder, symbol Device:R
Connections:
- net +3V3: now also U7.5 (SDO), R?.1, R?.1
- net I2C_SCL: now also R?.2
- net I2C_SDA: now also R?.2
Changed lines of the file:
@@
 Text Label 3150 6400 0    50   ~ 0
 TRIAC_W
+$Comp
+L Device:R R?
+U 1 1 5FBF57DD
+P 8000 5250
+F 0 "R?" V 7793 5250 50  0000 C CNN
+F 1 "180" V 7884 5250 50  0000 C CNN
+F 2 "Resistor_SMD:R_0805_2012Metric_Pad1.20x1.40mm_HandSolder" V 7930 5250 50  0001 C CNN
+F 3 "~" H 8000 5250 50  0001 C CNN
+F 4 "RT0805FRE07180RL" V 8000 5250 50  0001 C CNN "Part"
+	1    8000 5250
+	1    0    0    -1
+$EndComp
+$Comp
+L Device:R R?
+U 1 1 5FC004B4
+P 8350 5250
+F 0 "R?" V 8143 5250 50  0000 C CNN
+F 1 "180" V 8234 5250 50  0000 C CNN
+F 2 "Resistor_SMD:R_0805_2012Metric_Pad1.20x1.40mm_HandSolder" V 8280 5250 50  0001 C CNN
+F 3 "~" H 8350 5250 50  0001 C CNN
+F 4 "RT0805FRE07180RL" V 8350 5250 50  0001 C CNN "Part"
+	1    8350 5250
+	1    0    0    -1
+$EndComp
+Wire Wire Line
+	7600 5650 8350 5650
+Wire Wire Line
+	8350 5650 8350 5400
+Wire Wire Line
+	7600 5450 8000 5450
+Wire Wire Line
+	8000 5450 8000 5400
+Wire Wire Line
+	7100 4550 7600 4550
+Wire Wire Line
+	8000 4550 8000 5100
+Connection ~ 7100 4550
+Wire Wire Line
+	8000 4550 8350 4550
+Wire Wire Line
+	8350 4550 8350 5100
+Connection ~ 8000 4550
+Wire Wire Line
+	7600 5250 7600 4550
+Connection ~ 7600 4550
+Wire Wire Line
+	7600 4550 8000 4550
 $EndSCHEMATC

Commit message: Changed a few things around for better placement
Parts:
- removed SW3: 1825232-1, footprints:1825232-1, symbol 2020-11-02_17-45-18:1825232-1
- added Q2: 2N7002, digikey-footprints:SOT-23-3, symbol dk_Transistors-FETs-MOSFETs-Single:2N7002
- added R3: 10K, Resistor_SMD:R_0805_2012Metric_Pad1.20x1.40mm_HandSolder, symbol Device:R
- J7: footprint Connector_PinSocket_2.54mm:PinSocket_1x05_P2.54mm_Vertical -> Connector_PinSocket_2.54mm:PinSocket_1x03_P2.54mm_Vertical; symbol Connector_Generic:Conn_01x05 -> Connector_Generic:Conn_01x03
- R4, R5: renamed from R?; value 180 -> 10K
- R9: value 20K -> 10K
Connections:
- net EN is gone; now on net +VDC: U3.3 (EN)
- net +3V3: now also J4.2 (Pin_2), R3.2; no longer J4.3 (Pin_3), Q1.1 (C)
- net +5V: now also J7.3 (Pin_3), Q2.3 (D); no longer J3.4 (Pin_4), J7.4 (Pin_4)
- net C_TERM: now also J11.5; no longer J11.4
- net GND: now also J7.1 (Pin_1); no longer J7.2 (Pin_2)
- net G_TERM: now also J11.4; no longer J11.1
- net I2C_SCL: now also U1.36 (IO22); no longer U1.37 (IO23)
- net I2C_SDA: now also U1.37 (IO23); no longer U1.36 (IO22)
- net PIR: now also J7.2 (Pin_2); no longer J7.3 (Pin_3)
- net RC_TERM: now also J11.1; no longer J11.2
- net TRIAC_G: now also U1.10 (IO25); no longer U1.9 (IO33)
- net TRIAC_W: now also U1.8 (IO32); no longer U1.10 (IO25)
- net TRIAC_Y: now also U1.9 (IO33); no longer U1.8 (IO32)
- net W_TERM: now also J11.2; no longer J11.5
- net DISP_EN: now reaches U1.11 (IO26)
- net DISP_EN: now also Q2.1 (G)
- new net: Q1.1 (C), R3.1
- new net: J3.4 (Pin_4), Q2.2 (S)
Changed lines of the file:
@@
 $EndComp
 Text Label 3150 6200 2    50   ~ 0
-I2C_SDA
+I2C_SCL
 Wire Wire Line
 	2500 6200 3150 6200
@@
 	3900 950  3900 900
 Connection ~ 3900 900
-Wire Wire Line
-	3900 900  4250 900
 Wire Wire Line
 	2500 950  2500 900
@@
 PHOTO
 Text Label 3150 6700 2    50   ~ 0
-TRIAC_Y
+TRIAC_W
 Text Label 5150 1600 3    50   ~ 0
 ~ESP_RESET
@@
 $EndComp
 Wire Wire Line
-	3750 4650 4300 4650
-Wire Wire Line
 	4300 4350 4200 4350
 Wire Wire Line
@@
 	-1   0    0    1
 $EndComp
-Wire Wire Line
-	3750 4550 3750 4650
 $Comp
 L Switch:SW_Push SW2
@@
 	5500 1200 5500 1250
 $Comp
-L Connector_Generic:Conn_01x05 J7
+L Connector_Generic:Conn_01x03 J7
 U 1 1 6247059E
 P 5250 5750
 F 0 "J7" H 5168 5325 50  0000 C CNN
 F 1 "PIR" H 5168 5416 50  0000 C CNN
-F 2 "Connector_PinSocket_2.54mm:PinSocket_1x05_P2.54mm_Vertical" H 5250 5750 50  0001 C CNN
+F 2 "Connector_PinSocket_2.54mm:PinSocket_1x03_P2.54mm_Vertical" H 5250 5750 50  0001 C CNN
 F 3 "~" H 5250 5750 50  0001 C CNN
 	1    5250 5750
@@
 	5050 4600 4900 4600
 Wire Wire Line
-	4900 4600 4900 4350
-Wire Wire Line
 	5050 4900 4900 4900
 Wire Wire Line
@@
 L power:+5V #PWR0103
 U 1 1 601FC7D8
-P 4900 4350
-F 0 "#PWR0103" H 4900 4200 50  0001 C CNN
-F 1 "+5V" H 4915 4523 50  0000 C CNN
-F 2 "" H 4900 4350 50  0001 C CNN
-F 3 "" H 4900 4350 50  0001 C CNN
-	1    4900 4350
+P 5300 3600
+F 0 "#PWR0103" H 5300 3450 50  0001 C CNN
+F 1 "+5V" H 5315 3773 50  0000 C CNN
+F 2 "" H 5300 3600 50  0001 C CNN
+F 3 "" H 5300 3600 50  0001 C CNN
+	1    5300 3600
 	1    0    0    -1
 $EndComp
@@
 	2500 6900 3150 6900
 Text Label 3150 6800 2    50   ~ 0
-TRIAC_G
+TRIAC_Y
 Text Label 3150 6900 2    50   ~ 0
 PHOTO
 Text Label 3150 6300 0    50   ~ 0
-I2C_SCL
+I2C_SDA
 $Comp
 L Mechanical:MountingHole_Pad H2
@@
 	2500 6300 3150 6300
 Text Label 1400 8300 0    50   ~ 0
-C_TERM
+G_TERM
 Text Label 1400 8000 0    50   ~ 0
-G_TERM
+RC_TERM
 Text Label 1400 8100 0    50   ~ 0
-RC_TERM
+W_TERM
 Text Label 1400 8200 0    50   ~ 0
 Y_TERM
@@
 $EndComp
 Text Label 1400 8400 0    50   ~ 0
-W_TERM
+C_TERM
 Wire Wire Line
 	1400 8400 1650 8400
@@
 P 2850 8800
 F 0 "R9" H 2780 8754 50  0000 R CNN
-F 1 "20K" H 2780 8845 50  0000 R CNN
+F 1 "10K" H 2780 8845 50  0000 R CNN
 F 2 "Resistor_SMD:R_0805_2012Metric_Pad1.20x1.40mm_HandSolder" V 2780 8800 50  0001 C CNN
 F 3 "~" H 2850 8800 50  0001 C CNN
@@
 L power:+3.3V #PWR0105
 U 1 1 602B12AB
-P 2850 8150
-F 0 "#PWR0105" H 2850 8000 50  0001 C CNN
-F 1 "+3.3V" H 2865 8323 50  0000 C CNN
-F 2 "" H 2850 8150 50  0001 C CNN
-F 3 "" H 2850 8150 50  0001 C CNN
-	1    2850 8150
+P 2850 7850
+F 0 "#PWR0105" H 2850 7700 50  0001 C CNN
+F 1 "+3.3V" H 2865 8023 50  0000 C CNN
+F 2 "" H 2850 7850 50  0001 C CNN
+F 3 "" H 2850 7850 50  0001 C CNN
+	1    2850 7850
 	1    0    0    -1
 $EndComp
@@
 Wire Wire Line
 	5150 1300 5150 1500
-Text Label 4250 1100 0    50   ~ 0
-EN
-Text Label 4850 2900 0    50   ~ 0
-EN
-$Comp
-L 2020-11-02_17-45-18:1825232-1 SW3
-U 1 1 60A95A6A
-P 3250 2800
-F 0 "SW3" H 4050 3187 60  0000 C CNN
-F 1 "1825232-1" H 4050 3081 60  0000 C CNN
-F 2 "footprints:1825232-1" H 4050 3040 60  0001 C CNN
-F 3 "" H 3250 2800 60  0000 C CNN
-	1    3250 2800
-	1    0    0    -1
-$EndComp
 Wire Wire Line
 	2950 900  3450 900
-Wire Wire Line
-	4850 2800 4850 2650
-$Comp
-L power:+VDC #PWR0108
-U 1 1 60B2A0DC
-P 4850 2650
-F 0 "#PWR0108" H 4850 2550 50  0001 C CNN
-F 1 "+VDC" H 4850 2925 50  0000 C CNN
-F 2 "" H 4850 2650 50  0001 C CNN
-F 3 "" H 4850 2650 50  0001 C CNN
-	1    4850 2650
-	1    0    0    -1
-$EndComp
 Wire Wire Line
 	2850 8550 2850 8650
@@
 	2500 6400 3150 6400
 Text Label 3150 6400 0    50   ~ 0
-TRIAC_W
-$Comp
-L Device:R R?
+TRIAC_G
+$Comp
+L Device:R R4
 U 1 1 5FBF57DD
 P 8000 5250
-F 0 "R?" V 7793 5250 50  0000 C CNN
-F 1 "180" V 7884 5250 50  0000 C CNN
+F 0 "R4" V 7793 5250 50  0000 C CNN
+F 1 "10K" V 7884 5250 50  0000 C CNN
 F 2 "Resistor_SMD:R_0805_2012Metric_Pad1.20x1.40mm_HandSolder" V 7930 5250 50  0001 C CNN
 F 3 "~" H 8000 5250 50  0001 C CNN
@@
 $EndComp
 $Comp
-L Device:R R?
+L Device:R R5
 U 1 1 5FC004B4
 P 8350 5250
-F 0 "R?" V 8143 5250 50  0000 C CNN
-F 1 "180" V 8234 5250 50  0000 C CNN
+F 0 "R5" V 8143 5250 50  0000 C CNN
+F 1 "10K" V 8234 5250 50  0000 C CNN
 F 2 "Resistor_SMD:R_0805_2012Metric_Pad1.20x1.40mm_HandSolder" V 8280 5250 50  0001 C CNN
 F 3 "~" H 8350 5250 50  0001 C CNN
@@
 Wire Wire Line
 	7600 4550 8000 4550
+$Comp
+L Device:R R3
+U 1 1 5FDB81A5
+P 2850 8000
+F 0 "R3" H 2780 7954 50  0000 R CNN
+F 1 "10K" H 2780 8045 50  0000 R CNN
+F 2 "Resistor_SMD:R_0805_2012Metric_Pad1.20x1.40mm_HandSolder" V 2780 8000 50  0001 C CNN
+F 3 "~" H 2850 8000 50  0001 C CNN
+F 4 "RC0805FR-07100KL" H 2850 8000 50  0001 C CNN "Part"
+	1    2850 8000
+	-1   0    0    1
+$EndComp
+$Comp
+L dk_Transistors-FETs-MOSFETs-Single:2N7002 Q2
+U 1 1 5FE3E266
+P 5300 3800
+F 0 "Q2" H 5408 3853 60  0000 L CNN
+F 1 "2N7002" H 5408 3747 60  0000 L CNN
+F 2 "digikey-footprints:SOT-23-3" H 5500 4000 60  0001 L CNN
+F 3 "https://www.onsemi.com/pub/Collateral/NDS7002A-D.PDF" H 5500 4100 60  0001 L CNN
+F 4 "2N7002NCT-ND" H 5500 4200 60  0001 L CNN "Digi-Key_PN"
+F 5 "2N7002" H 5500 4300 60  0001 L CNN "MPN"
+F 6 "Discrete Semiconductor Products" H 5500 4400 60  0001 L CNN "Category"
+F 7 "Transistors - FETs, MOSFETs - Single" H 5500 4500 60  0001 L CNN "Family"
+F 8 "https://www.onsemi.com/pub/Collateral/NDS7002A-D.PDF" H 5500 4600 60  0001 L CNN "DK_Datasheet_Link"
+F 9 "/product-detail/en/on-semiconductor/2N7002/2N7002NCT-ND/244664" H 5500 4700 60  0001 L CNN "DK_Detail_Page"
+F 10 "MOSFET N-CH 60V 115MA SOT-23" H 5500 4800 60  0001 L CNN "Description"
+F 11 "ON Semiconductor" H 5500 4900 60  0001 L CNN "Manufacturer"
+F 12 "Active" H 5500 5000 60  0001 L CNN "Status"
+	1    5300 3800
+	1    0    0    -1
+$EndComp
+Wire Wire Line
+	13300 5900 13300 950
+Wire Wire Line
+	13300 950  20650 950
+Wire Wire Line
+	5000 3900 4850 3900
+Text Label 4850 3900 0    50   ~ 0
+DISP_EN
+Wire Wire Line
+	5300 4000 4900 4000
+Wire Wire Line
+	4900 4000 4900 4600
+Wire Wire Line
+	2500 6500 3150 6500
+Text Label 3150 6500 0    50   ~ 0
+DISP_EN
+Wire Wire Line
+	4250 1100 4150 1100
+Wire Wire Line
+	4150 1100 4150 900
+Wire Wire Line
+	3900 900  4150 900
+Wire Wire Line
+	4150 900  4250 900
+Connection ~ 4150 900
+Wire Wire Line
+	3750 4750 4300 4750
+Wire Wire Line
+	3750 4550 3750 4750
 $EndSCHEMATC

Commit message: Moved 680 to bottom and switched ldo to buck
Parts:
- removed C13: 220 uF, Capacitor_SMD:CP_Elec_8x10, symbol Device:CP
- removed C9: 10 uF, Capacitor_SMD:CP_Elec_5x5.8, symbol Device:CP
- removed D3: STATUS, LED_SMD:LED_1206_3216Metric_ReverseMount_Hole1.8x2.4mm, symbol Device:LED
- removed R12: 1K6, Resistor_SMD:R_0805_2012Metric_Pad1.20x1.40mm_HandSolder, symbol Device:R
- removed R15: 120, Resistor_SMD:R_0805_2012Metric_Pad1.20x1.40mm_HandSolder, symbol Device:R
- removed U4: LD1086DT33TR, Package_TO_SOT_SMD:TO-252-2, symbol Regulator_Linear:LD1086DT33TR
- added C10: 10 uF, Capacitor_SMD:C_0805_2012Metric, symbol Device:C
- added C9: 10 uf, Capacitor_SMD:C_0805_2012Metric, symbol Device:C
- added R6: 523k, Resistor_SMD:R_0805_2012Metric_Pad1.20x1.40mm_HandSolder, symbol Device:R
- added R7: 169k, Resistor_SMD:R_0805_2012Metric_Pad1.20x1.40mm_HandSolder, symbol Device:R
- added R8: 8K2, Resistor_SMD:R_0805_2012Metric_Pad1.20x1.40mm_HandSolder, symbol Device:R
- added SW3: 1825232-1, footprints:1825232-1, symbol 2020-11-02_17-45-18:1825232-1
- added U2: TPS82084SILR, footprints:Texas_Instruments-SIL0008C-0-0-MFG, symbol eec:TPS82084SILR
- C12: value 10 uF -> 220 uF; footprint Capacitor_SMD:CP_Elec_5x5.8 -> Capacitor_SMD:CP_Elec_8x10; Part EEE-HP0J100R -> EEE-HB0J221AP
- D2: value 3V3 -> 3V
- J7: footprint Connector_PinSocket_2.54mm:PinSocket_1x03_P2.54mm_Vertical -> Connector_PinHeader_2.54mm:PinHeader_1x03_P2.54mm_Vertical
- R3: value 10K -> 499k; Part RC0805FR-07100KL -> CRCW0805499KFKEA
- R4, R5: value 10K -> 3.3k
- R9: value 10K -> 4K
Connections:
- net +3V3: now also Q1.1 (C), R3.1, U7.2 (CSB), C10.1, R6.1, R8.2, U2.8 (VOUT); no longer R3.2
- net +5V: now also C9.1, SW3.3, U2.1 (EN), U2.3 (VIN), U2.4 (VIN); no longer C14.1, C15.1, C16.1, L1.2, R10.1, R16.2
- net GND: now also C10.2, C9.2, R7.2, U2.5 (GND), U2.6 (GND), U2.9 (EXPOSED_THERMAL_PAD)
- net ~ESP_RESET: now also JP1.1 (Pin_1); no longer JP1.2 (Pin_2)
- net at D2.2 (A): now also R8.1
- net at U3.4 (PG): no longer JP1.1 (Pin_1)
- net STATUS: no longer names the net of U1.29 (IO5)
- new net: JP1.2 (Pin_2), R3.2, U2.2 (PG)
- new net: R6.2, R7.1, U2.7 (FB)
- new net 5V_Switch: C14.1, C15.1, C16.1, L1.2, R10.1, R16.2, SW3.2
Other:
- moved on the sheet: D4, JP1, R16

Commit message: Moved 680 to other side of board
Connections:
- net I2C_SCL: now also U1.37 (IO23); no longer U1.36 (IO22)
- net I2C_SDA: now also U1.36 (IO22); no longer U1.37 (IO23)
Changed lines of the file:
@@
 MODE
 Text Label 3150 6200 2    50   ~ 0
-I2C_SCL
+I2C_SDA
 Wire Wire Line
 	2500 6200 3150 6200
@@
 PHOTO
 Text Label 3150 6300 0    50   ~ 0
-I2C_SDA
+I2C_SCL
 $Comp
 L Mechanical:MountingHole_Pad H2
